Commit message: 🌱init commit: 初期コミット

File: orne_box_description/urdf/orne_box.gazebo.xacro (robot description, xacro)
@@ -76,5 +76,5 @@
     </gazebo>
     <!-- imu -->
-    <gazebo reference="imu_link">
+    <!-- <gazebo reference="imu_link">
       <sensor type="imu" name="imu">
         <plugin filename="libgazebo_ros_imu_sensor.so" name="imu_plugin">
@@ -143,5 +143,5 @@
       </sensor>
       <material>Gazebo/Green</material>
-    </gazebo>
+    </gazebo> -->
     <!-- hokuyo -->
     <gazebo reference="hokuyo_link">

File: orne_box_description/urdf/orne_box.urdf.xacro (robot description, xacro)
@@ -11,5 +11,5 @@
   <xacro:include filename="$(find orne_box_description)/urdf/joints/caster_swivel_joint.urdf.xacro"/>
   <xacro:include filename="$(find orne_box_description)/urdf/joints/wheel_joint.urdf.xacro"/>
-  <xacro:include filename="$(find orne_box_description)/urdf/sensors/imu.urdf.xacro"/>
+  <!-- <xacro:include filename="$(find orne_box_description)/urdf/sensors/imu.urdf.xacro"/> -->
   <xacro:include filename="$(find orne_box_description)/urdf/sensors/hokuyo.urdf.xacro"/>
   <!-- Setting for base -->
@@ -48,14 +48,14 @@
     <origin xyz="0.23 0.0 0.270" rpy="${-PI} 0 ${PI/2}"/>
   </xacro:sensor_imu> -->
-  <xacro:sensor_imu name="imu" parent="base_link" size="0.05 0.05 0.05">
+  <!-- <xacro:sensor_imu name="imu" parent="base_link" size="0.05 0.05 0.05">
     <origin xyz="0.23 0.0 0.270" rpy="0 0 0"/>
     <origin_child xyz="0.0 0.0 0.0" rpy="0 0 0"/>
-  </xacro:sensor_imu>
+  </xacro:sensor_imu> -->
   <!-- Setting for 2D-LiDAR -->
   <xacro:sensor_hokuyo name="hokuyo" parent="base_link" size="0.05 0.05 0.05">
-    <origin xyz="0.374295 0 0.2185" rpy="${-PI} 0 0"/>
+    <origin xyz="0.374295 0 0.2185" rpy="0 0 0"/>
   </xacro:sensor_hokuyo>
-  <xacro:sensor_hokuyo name="mirror_lidar" parent="base_link" size="0.05 0.05 0.05">
-    <origin xyz="0.43 0.0 0.34" rpy="0 0.314 0"/>
-  </xacro:sensor_hokuyo>
+  <!-- <xacro:sensor_hokuyo name="mirror_lidar" parent="base_link" size="0.05 0.05 0.05"> -->
+    <!-- <origin xyz="0.43 0.0 0.34" rpy="0 0.314 0"/> -->
+  <!-- </xacro:sensor_hokuyo> -->
 </robot>
