Commit message: 🔧modify: rfans位置conflict修正

File: orne_box_description/urdf/orne_box_3d_lidar_rfans.urdf.xacro (robot description, xacro)
@@ -8,5 +8,6 @@
     <!-- Setting for 3D-LiDAR -->
     <xacro:VLP-16 parent="base_link" name="surestar" topic="/rfans_points" organize_cloud="false" hz="10" samples="440" gpu="false">
-      <origin xyz="0.23 0 0.40" rpy="0 0 0"/>
+      <!-- <origin xyz="0.23 0 0.40" rpy="0 0 3.14"/> -->
+      <origin xyz="-0.1 0 0.6" rpy="0 0 3.14"/>
     </xacro:VLP-16>
   </xacro:if>
